File: Hardware/file5CDA5614.sch (KiCad schematic (older format))
At the start: 17 parts

Commit message: Assigned all footprints.
Still need to pick and check FET footprint, pick pot.
Parts:
- C14, C15, C16, C17, C18, C19: renamed from C?; footprint (none) -> Capacitor_SMD:C_0603_1608Metric
- Q1, Q2, Q3, Q4: renamed from Q?; footprint (none) -> Package_TO_SOT_SMD:TO-252-2
- R10, R11, R12, R13, R8, R9: renamed from R?; footprint (none) -> Resistor_SMD:R_0603_1608Metric
- gave numbers to parts that had none: 1

Commit message: Started moving components around on PCB.
Parts:
- U6: footprint (none) -> Package_SO:HTSSOP-24-1EP_4.4x7.8mm_P0.65mm_EP3.4x7.8mm_Mask2.4x4.68mm
Changed lines of the file:
@@
 $Descr A4 11693 8268
 encoding utf-8
-Sheet 2 3
+Sheet 3 3
 Title ""
 Date ""
@@
 AR Path="/5CDCD2BF/5CDB0CF0" Ref="U?"  Part="1"
 AR Path="/5D4DF0EE/5CDB0CF0" Ref="U7"  Part="1"
-F 0 "U6" H 5200 3265 50  0000 C CNN
+F 0 "U7" H 5200 3265 50  0000 C CNN
 F 1 "A4940KLPTR-T" H 5200 3174 50  0000 C CNN
-F 2 "" H 5100 2850 50  0001 C CNN
+F 2 "Package_SO:HTSSOP-24-1EP_4.4x7.8mm_P0.65mm_EP3.4x7.8mm_Mask2.4x4.68mm" H 5100 2850 50  0001 C CNN
 F 3 "" H 5100 2850 50  0001 C CNN
 	1    5200 2850
@@
 AR Path="/5CDCD2BF/5CDB0CF6" Ref="Q?"  Part="1"
 AR Path="/5D4DF0EE/5CDB0CF6" Ref="Q5"  Part="1"
-F 0 "Q1" H 8606 2496 50  0000 L CNN
+F 0 "Q5" H 8606 2496 50  0000 L CNN
 F 1 "Q_NMOS_DGS" H 8606 2405 50  0000 L CNN
 F 2 "Package_TO_SOT_SMD:TO-252-2" H 8600 2550 50  0001 C CNN
@@
 AR Path="/5CDCD2BF/5CDB0CFC" Ref="Q?"  Part="1"
 AR Path="/5D4DF0EE/5CDB0CFC" Ref="Q6"  Part="1"
-F 0 "Q2" H 8606 3146 50  0000 L CNN
+F 0 "Q6" H 8606 3146 50  0000 L CNN
 F 1 "Q_NMOS_DGS" H 8606 3055 50  0000 L CNN
 F 2 "Package_TO_SOT_SMD:TO-252-2" H 8600 3200 50  0001 C CNN
@@
 AR Path="/5CDCD2BF/5CDB0D02" Ref="R?"  Part="1"
 AR Path="/5D4DF0EE/5CDB0D02" Ref="R16"  Part="1"
-F 0 "R10" V 7745 2450 50  0000 C CNN
+F 0 "R16" V 7745 2450 50  0000 C CNN
 F 1 "27" V 7836 2450 50  0000 C CNN
 F 2 "Resistor_SMD:R_0603_1608Metric" V 7990 2440 50  0001 C CNN
@@
 AR Path="/5CDCD2BF/5CDB0D08" Ref="R?"  Part="1"
 AR Path="/5D4DF0EE/5CDB0D08" Ref="R17"  Part="1"
-F 0 "R11" V 7745 3100 50  0000 C CNN
+F 0 "R17" V 7745 3100 50  0000 C CNN
 F 1 "27" V 7836 3100 50  0000 C CNN
 F 2 "Resistor_SMD:R_0603_1608Metric" V 7990 3090 50  0001 C CNN
@@
 AR Path="/5CDCD2BF/5CDB0D0E" Ref="C?"  Part="1"
 AR Path="/5D4DF0EE/5CDB0D0E" Ref="C22"  Part="1"
-F 0 "C16" V 6200 2600 50  0000 C CNN
+F 0 "C22" V 6200 2600 50  0000 C CNN
 F 1 "0.1u" V 6200 2850 50  0000 C CNN
 F 2 "Capacitor_SMD:C_0603_1608Metric" H 6300 2700 50  0001 C CNN
@@
 AR Path="/5CDCD2BF/5CDB0D14" Ref="C?"  Part="1"
 AR Path="/5D4DF0EE/5CDB0D14" Ref="C23"  Part="1"
-F 0 "C17" V 6250 2750 50  0000 C CNN
+F 0 "C23" V 6250 2750 50  0000 C CNN
 F 1 "1u" V 6250 3000 50  0000 C CNN
 F 2 "Capacitor_SMD:C_0603_1608Metric" H 6300 2850 50  0001 C CNN
@@
 AR Path="/5CDCD2BF/5CDB0D1A" Ref="C?"  Part="1"
 AR Path="/5D4DF0EE/5CDB0D1A" Ref="C24"  Part="1"
-F 0 "C18" V 6250 3200 50  0000 C CNN
+F 0 "C24" V 6250 3200 50  0000 C CNN
 F 1 "1u" V 6250 3400 50  0000 C CNN
 F 2 "Capacitor_SMD:C_0603_1608Metric" H 6300 3300 50  0001 C CNN
@@
 AR Path="/5CDCD2BF/5CDB0D20" Ref="C?"  Part="1"
 AR Path="/5D4DF0EE/5CDB0D20" Ref="C25"  Part="1"
-F 0 "C19" V 6350 3850 50  0000 C CNN
+F 0 "C25" V 6350 3850 50  0000 C CNN
 F 1 "1u" V 6350 3650 50  0000 C CNN
 F 2 "Capacitor_SMD:C_0603_1608Metric" H 6300 3750 50  0001 C CNN
@@
 AR Path="/5CDCD2BF/5CDB0D28" Ref="#PWR?"  Part="1"
 AR Path="/5D4DF0EE/5CDB0D28" Ref="#PWR074"  Part="1"
-F 0 "#PWR060" H 5950 2250 50  0001 C CNN
+F 0 "#PWR074" H 5950 2250 50  0001 C CNN
 F 1 "VBUS" H 5965 2573 50  0000 C CNN
 F 2 "" H 5950 2400 50  0001 C CNN
@@
 AR Path="/5CDCD2BF/5CDB0D51" Ref="#PWR?"  Part="1"
 AR Path="/5D4DF0EE/5CDB0D51" Ref="#PWR075"  Part="1"
-F 0 "#PWR061" H 6550 2450 50  0001 C CNN
+F 0 "#PWR075" H 6550 2450 50  0001 C CNN
 F 1 "GND" V 6555 2572 50  0000 R CNN
 F 2 "" H 6550 2700 50  0001 C CNN
@@
 AR Path="/5CDCD2BF/5CDB0D59" Ref="Q?"  Part="1"
 AR Path="/5D4DF0EE/5CDB0D59" Ref="Q7"  Part="1"
-F 0 "Q3" H 8606 4296 50  0000 L CNN
+F 0 "Q7" H 8606 4296 50  0000 L CNN
 F 1 "Q_NMOS_DGS" H 8606 4205 50  0000 L CNN
 F 2 "Package_TO_SOT_SMD:TO-252-2" H 8600 4350 50  0001 C CNN
@@
 AR Path="/5CDCD2BF/5CDB0D5F" Ref="Q?"  Part="1"
 AR Path="/5D4DF0EE/5CDB0D5F" Ref="Q8"  Part="1"
-F 0 "Q4" H 8606 4946 50  0000 L CNN
+F 0 "Q8" H 8606 4946 50  0000 L CNN
 F 1 "Q_NMOS_DGS" H 8606 4855 50  0000 L CNN
 F 2 "Package_TO_SOT_SMD:TO-252-2" H 8600 5000 50  0001 C CNN
@@
 AR Path="/5CDCD2BF/5CDB0D65" Ref="R?"  Part="1"
 AR Path="/5D4DF0EE/5CDB0D65" Ref="R18"  Part="1"
-F 0 "R12" V 7745 4250 50  0000 C CNN
+F 0 "R18" V 7745 4250 50  0000 C CNN
 F 1 "27" V 7836 4250 50  0000 C CNN
 F 2 "Resistor_SMD:R_0603_1608Metric" V 7990 4240 50  0001 C CNN
@@
 AR Path="/5CDCD2BF/5CDB0D6B" Ref="R?"  Part="1"
 AR Path="/5D4DF0EE/5CDB0D6B" Ref="R19"  Part="1"
-F 0 "R13" V 7745 4900 50  0000 C CNN
+F 0 "R19" V 7745 4900 50  0000 C CNN
 F 1 "27" V 7836 4900 50  0000 C CNN
 F 2 "Resistor_SMD:R_0603_1608Metric" V 7990 4890 50  0001 C CNN
@@
 AR Path="/5CDCD2BF/5CDB0D89" Ref="#PWR?"  Part="1"
 AR Path="/5D4DF0EE/5CDB0D89" Ref="#PWR077"  Part="1"
-F 0 "#PWR063" H 8500 3050 50  0001 C CNN
+F 0 "#PWR077" H 8500 3050 50  0001 C CNN
 F 1 "GND" H 8505 3127 50  0000 C CNN
 F 2 "" H 8500 3300 50  0001 C CNN
@@
 AR Path="/5CDCD2BF/5CDB0D95" Ref="#PWR?"  Part="1"
 AR Path="/5D4DF0EE/5CDB0D95" Ref="#PWR079"  Part="1"
-F 0 "#PWR065" H 8500 4850 50  0001 C CNN
+F 0 "#PWR079" H 8500 4850 50  0001 C CNN
 F 1 "GND" H 8505 4927 50  0000 C CNN
 F 2 "" H 8500 5100 50  0001 C CNN
@@
 AR Path="/5CDCD2BF/5CDB0D9B" Ref="#PWR?"  Part="1"
 AR Path="/5D4DF0EE/5CDB0D9B" Ref="#PWR076"  Part="1"
-F 0 "#PWR062" H 8500 2050 50  0001 C CNN
+F 0 "#PWR076" H 8500 2050 50  0001 C CNN
 F 1 "VBUS" H 8515 2373 50  0000 C CNN
 F 2 "" H 8500 2200 50  0001 C CNN
@@
 AR Path="/5CDCD2BF/5CDB0DA2" Ref="#PWR?"  Part="1"
 AR Path="/5D4DF0EE/5CDB0DA2" Ref="#PWR078"  Part="1"
-F 0 "#PWR064" H 8500 3850 50  0001 C CNN
+F 0 "#PWR078" H 8500 3850 50  0001 C CNN
 F 1 "VBUS" H 8515 4173 50  0000 C CNN
 F 2 "" H 8500 4000 50  0001 C CNN
@@
 AR Path="/5CDCD2BF/5CDB0DB9" Ref="#PWR?"  Part="1"
 AR Path="/5D4DF0EE/5CDB0DB9" Ref="#PWR073"  Part="1"
-F 0 "#PWR059" H 5900 4150 50  0001 C CNN
+F 0 "#PWR073" H 5900 4150 50  0001 C CNN
 F 1 "GND" H 5905 4227 50  0000 C CNN
 F 2 "" H 5900 4400 50  0001 C CNN
@@
 AR Path="/5CDCD2BF/5CDB0DC6" Ref="#PWR?"  Part="1"
 AR Path="/5D4DF0EE/5CDB0DC6" Ref="#PWR072"  Part="1"
-F 0 "#PWR058" H 5200 4150 50  0001 C CNN
+F 0 "#PWR072" H 5200 4150 50  0001 C CNN
 F 1 "GND" H 5205 4227 50  0000 C CNN
 F 2 "" H 5200 4400 50  0001 C CNN
@@
 AR Path="/5CDCD2BF/5CDB0DCC" Ref="#PWR?"  Part="1"
 AR Path="/5D4DF0EE/5CDB0DCC" Ref="#PWR071"  Part="1"
-F 0 "#PWR057" H 4500 4150 50  0001 C CNN
+F 0 "#PWR071" H 4500 4150 50  0001 C CNN
 F 1 "GND" H 4505 4227 50  0000 C CNN
 F 2 "" H 4500 4400 50  0001 C CNN
@@
 AR Path="/5CDCD2BF/5CDB0DD5" Ref="#PWR?"  Part="1"
 AR Path="/5D4DF0EE/5CDB0DD5" Ref="#PWR070"  Part="1"
-F 0 "#PWR056" H 4250 4150 50  0001 C CNN
+F 0 "#PWR070" H 4250 4150 50  0001 C CNN
 F 1 "GND" H 4255 4227 50  0000 C CNN
 F 2 "" H 4250 4400 50  0001 C CNN
@@
 AR Path="/5CDCD2BF/5CDB0DDB" Ref="R?"  Part="1"
 AR Path="/5D4DF0EE/5CDB0DDB" Ref="R15"  Part="1"
-F 0 "R9" V 4245 4050 50  0000 C CNN
+F 0 "R15" V 4245 4050 50  0000 C CNN
 F 1 "82k" V 4336 4050 50  0000 C CNN
 F 2 "Resistor_SMD:R_0603_1608Metric" V 4490 4040 50  0001 C CNN
@@
 AR Path="/5CDCD2BF/5CDB0DE9" Ref="#PWR?"  Part="1"
 AR Path="/5D4DF0EE/5CDB0DE9" Ref="#PWR066"  Part="1"
-F 0 "#PWR052" H 3300 2450 50  0001 C CNN
+F 0 "#PWR066" H 3300 2450 50  0001 C CNN
 F 1 "+5V" H 3315 2773 50  0000 C CNN
 F 2 "" H 3300 2600 50  0001 C CNN
@@
 AR Path="/5CDCD2BF/5CDB0DEF" Ref="C?"  Part="1"
 AR Path="/5D4DF0EE/5CDB0DEF" Ref="C21"  Part="1"
-F 0 "C15" H 3792 2946 50  0000 L CNN
+F 0 "C21" H 3792 2946 50  0000 L CNN
 F 1 "10u" H 3792 2855 50  0000 L CNN
 F 2 "Capacitor_SMD:C_0603_1608Metric" H 3700 2900 50  0001 C CNN
@@
 AR Path="/5CDCD2BF/5CDB0DFE" Ref="C?"  Part="1"
 AR Path="/5D4DF0EE/5CDB0DFE" Ref="C20"  Part="1"
-F 0 "C14" H 3392 2946 50  0000 L CNN
+F 0 "C20" H 3392 2946 50  0000 L CNN
 F 1 "0.1u" H 3392 2855 50  0000 L CNN
 F 2 "Capacitor_SMD:C_0603_1608Metric" H 3300 2900 50  0001 C CNN
@@
 AR Path="/5CDCD2BF/5CDB0E08" Ref="#PWR?"  Part="1"
 AR Path="/5D4DF0EE/5CDB0E08" Ref="#PWR067"  Part="1"
-F 0 "#PWR053" H 3300 2750 50  0001 C CNN
+F 0 "#PWR067" H 3300 2750 50  0001 C CNN
 F 1 "GND" H 3305 2827 50  0000 C CNN
 F 2 "" H 3300 3000 50  0001 C CNN
@@
 AR Path="/5CDCD2BF/5CDB0E0E" Ref="#PWR?"  Part="1"
 AR Path="/5D4DF0EE/5CDB0E0E" Ref="#PWR069"  Part="1"
-F 0 "#PWR055" H 3700 2750 50  0001 C CNN
+F 0 "#PWR069" H 3700 2750 50  0001 C CNN
 F 1 "GND" H 3705 2827 50  0000 C CNN
 F 2 "" H 3700 3000 50  0001 C CNN
@@
 AR Path="/5CDA5615/5D4C02AF" Ref="R8"  Part="1"
 AR Path="/5D4DF0EE/5D4C02AF" Ref="R14"  Part="1"
-F 0 "R8" V 4000 3500 50  0000 L CNN
+F 0 "R14" V 4000 3500 50  0000 L CNN
 F 1 "10k" V 3900 3450 50  0000 L CNN
 F 2 "Resistor_SMD:R_0603_1608Metric" V 3840 3540 50  0001 C CNN
@@
 AR Path="/5CDA5615/5D4CA44D" Ref="#PWR054"  Part="1"
 AR Path="/5D4DF0EE/5D4CA44D" Ref="#PWR068"  Part="1"
-F 0 "#PWR054" H 3600 3400 50  0001 C CNN
+F 0 "#PWR068" H 3600 3400 50  0001 C CNN
 F 1 "+5V" H 3615 3723 50  0000 C CNN
 F 2 "" H 3600 3550 50  0001 C CNN

Commit message: Fixed small issues and started laying out H-bridge
Parts:
- removed Q1, Q2, Q3, Q4: Q_NMOS_DGS, Package_TO_SOT_SMD:TO-252-2, symbol Device:Q_NMOS_DGS
- added Q1, Q2, Q3, Q4: Q_NMOS_GDS, Package_TO_SOT_SMD:TO-252-2, symbol Device:Q_NMOS_GDS
