File: bumblebee-board/Bumblebee-dual-motor-driver.sch (KiCad schematic (older format))
At the start: 53 parts, among them J1 ICSP, J10 GND, J11 MOTOR1_A, J12 MOTOR1_B, J13 MOTOR2_A, J14 MOTOR2_B, J15 MAIN+, J16 MAIN-, J17 HEADER, J18 JST-XH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

Commit message: Bumblebee-board r2 ready to ship.
Connections:
- net +5V: now also U5.3 (OUT); no longer U5.1 (IN)
- net MOTOR1_PWM: now also U1.10 (PD6); no longer U1.1 (PD3)
- net MOTOR2_DIR: now also U1.1 (PD3); no longer U1.10 (PD6)
- net VBUS: now also U5.1 (IN); no longer U5.3 (OUT)
Changed lines of the file:
@@
 	1    0    0    -1
 $EndComp
-Text Label 2600 3250 2    50   ~ 0
-MOTOR1_PWM
-Wire Wire Line
-	2050 3250 2600 3250
 Text Label 2600 3450 2    50   ~ 0
 MOTOR2_PWM
@@
 	2050 3450 2600 3450
 Wire Wire Line
-	2050 3550 2600 3550
+	2050 3250 2600 3250
 Wire Wire Line
 	2050 3350 2600 3350
 Text Label 2600 3350 2    50   ~ 0
 MOTOR1_DIR
-Text Label 2600 3550 2    50   ~ 0
+Text Label 2600 3250 2    50   ~ 0
 MOTOR2_DIR
 Wire Wire Line
@@
 F 3 "https://www.recom-power.com/pdf/Innoline/R-78Exx-0.5.pdf" H 7950 3600 50  0001 C CNN
 	1    7950 3600
-	1    0    0    -1
+	-1   0    0    -1
 $EndComp
 $Comp
@@
 Text Label 2100 4700 2    50   ~ 0
 USB_PWR
+Wire Wire Line
+	2050 3550 2600 3550
+Text Label 2600 3550 2    50   ~ 0
+MOTOR1_PWM
 $EndSCHEMATC
