File: bumblebee-board/file5CDA5614.sch (KiCad schematic (older format))
At the start: 17 parts, among them Q1 Q_NMOS_GDS, Q2 Q_NMOS_GDS, Q3 Q_NMOS_GDS, Q4 Q_NMOS_GDS, U6 A4940KLPTR-T

Commit message: Bumblebee-board r2 ready to ship.
Parts:
- added R8: 27k, Resistor_SMD:R_0603_1608Metric, symbol Device:R_US
- renumbered R9 to R10, R10 to R11, R11 to R12, R12 to R13, R13 to R14, R8 to R9
Connections:
- net VBUS: now also R8.2
- net ~RESET: now also R8.1
