File: bumblebee-board/file5CDA5615.sch (KiCad schematic (older format))
At the start: 17 parts, among them Q5 Q_NMOS_GDS, Q6 Q_NMOS_GDS, Q7 Q_NMOS_GDS, Q8 Q_NMOS_GDS, U7 A4940KLPTR-T

Commit message: Bumblebee-board r2 ready to ship.
Parts:
- added R15: 27k, Resistor_SMD:R_0603_1608Metric, symbol Device:R_US
- renumbered R14 to R16, R15 to R17, R16 to R18, R17 to R19, R18 to R22, R19 to R23
Connections:
- net VBUS: now also R15.2
- net ~RESET: now also R15.1
Changed lines of the file:
@@
 AR Path="/5CDA5615/5CE7F856" Ref="R?"  Part="1"
 AR Path="/5CDCD2BF/5CE7F856" Ref="R?"  Part="1"
-AR Path="/5D4DF0EE/5CE7F856" Ref="R16"  Part="1"
-F 0 "R16" V 7645 2500 50  0000 C CNN
+AR Path="/5D4DF0EE/5CE7F856" Ref="R18"  Part="1"
+F 0 "R18" V 7645 2500 50  0000 C CNN
 F 1 "27" V 7736 2500 50  0000 C CNN
 F 2 "Resistor_SMD:R_0603_1608Metric" V 7890 2490 50  0001 C CNN
@@
 AR Path="/5CDA5615/5CE7F85C" Ref="R?"  Part="1"
 AR Path="/5CDCD2BF/5CE7F85C" Ref="R?"  Part="1"
-AR Path="/5D4DF0EE/5CE7F85C" Ref="R17"  Part="1"
-F 0 "R17" V 7645 3150 50  0000 C CNN
+AR Path="/5D4DF0EE/5CE7F85C" Ref="R19"  Part="1"
+F 0 "R19" V 7645 3150 50  0000 C CNN
 F 1 "27" V 7736 3150 50  0000 C CNN
 F 2 "Resistor_SMD:R_0603_1608Metric" V 7890 3140 50  0001 C CNN
@@
 AR Path="/5CDA5615/5CE7F891" Ref="#PWR?"  Part="1"
 AR Path="/5CDCD2BF/5CE7F891" Ref="#PWR?"  Part="1"
-AR Path="/5D4DF0EE/5CE7F891" Ref="#PWR0103"  Part="1"
-F 0 "#PWR0103" H 6450 2500 50  0001 C CNN
+AR Path="/5D4DF0EE/5CE7F891" Ref="#PWR0119"  Part="1"
+F 0 "#PWR0119" H 6450 2500 50  0001 C CNN
 F 1 "GND" V 6455 2622 50  0000 R CNN
 F 2 "" H 6450 2750 50  0001 C CNN
@@
 AR Path="/5CDA5615/5CE7F899" Ref="R?"  Part="1"
 AR Path="/5CDCD2BF/5CE7F899" Ref="R?"  Part="1"
-AR Path="/5D4DF0EE/5CE7F899" Ref="R18"  Part="1"
-F 0 "R18" V 7645 4300 50  0000 C CNN
+AR Path="/5D4DF0EE/5CE7F899" Ref="R22"  Part="1"
+F 0 "R22" V 7645 4300 50  0000 C CNN
 F 1 "27" V 7736 4300 50  0000 C CNN
 F 2 "Resistor_SMD:R_0603_1608Metric" V 7890 4290 50  0001 C CNN
@@
 AR Path="/5CDA5615/5CE7F89F" Ref="R?"  Part="1"
 AR Path="/5CDCD2BF/5CE7F89F" Ref="R?"  Part="1"
-AR Path="/5D4DF0EE/5CE7F89F" Ref="R19"  Part="1"
-F 0 "R19" V 7645 4950 50  0000 C CNN
+AR Path="/5D4DF0EE/5CE7F89F" Ref="R23"  Part="1"
+F 0 "R23" V 7645 4950 50  0000 C CNN
 F 1 "27" V 7736 4950 50  0000 C CNN
 F 2 "Resistor_SMD:R_0603_1608Metric" V 7890 4940 50  0001 C CNN
@@
 AR Path="/5CDA5615/5CE7F8AA" Ref="#PWR?"  Part="1"
 AR Path="/5CDCD2BF/5CE7F8AA" Ref="#PWR?"  Part="1"
-AR Path="/5D4DF0EE/5CE7F8AA" Ref="#PWR0104"  Part="1"
-F 0 "#PWR0104" H 8400 3100 50  0001 C CNN
+AR Path="/5D4DF0EE/5CE7F8AA" Ref="#PWR0120"  Part="1"
+F 0 "#PWR0120" H 8400 3100 50  0001 C CNN
 F 1 "GND" H 8405 3177 50  0000 C CNN
 F 2 "" H 8400 3350 50  0001 C CNN
@@
 AR Path="/5CDA5615/5CE7F8B0" Ref="#PWR?"  Part="1"
 AR Path="/5CDCD2BF/5CE7F8B0" Ref="#PWR?"  Part="1"
-AR Path="/5D4DF0EE/5CE7F8B0" Ref="#PWR0105"  Part="1"
-F 0 "#PWR0105" H 8400 4900 50  0001 C CNN
+AR Path="/5D4DF0EE/5CE7F8B0" Ref="#PWR0121"  Part="1"
+F 0 "#PWR0121" H 8400 4900 50  0001 C CNN
 F 1 "GND" H 8405 4977 50  0000 C CNN
 F 2 "" H 8400 5150 50  0001 C CNN
@@
 AR Path="/5CDA5615/5CE7F8B6" Ref="#PWR?"  Part="1"
 AR Path="/5CDCD2BF/5CE7F8B6" Ref="#PWR?"  Part="1"
-AR Path="/5D4DF0EE/5CE7F8B6" Ref="#PWR0106"  Part="1"
-F 0 "#PWR0106" H 8400 2100 50  0001 C CNN
+AR Path="/5D4DF0EE/5CE7F8B6" Ref="#PWR0122"  Part="1"
+F 0 "#PWR0122" H 8400 2100 50  0001 C CNN
 F 1 "VBUS" H 8415 2423 50  0000 C CNN
 F 2 "" H 8400 2250 50  0001 C CNN
@@
 AR Path="/5CDA5615/5CE7F8BD" Ref="#PWR?"  Part="1"
 AR Path="/5CDCD2BF/5CE7F8BD" Ref="#PWR?"  Part="1"
-AR Path="/5D4DF0EE/5CE7F8BD" Ref="#PWR0107"  Part="1"
-F 0 "#PWR0107" H 8400 3900 50  0001 C CNN
+AR Path="/5D4DF0EE/5CE7F8BD" Ref="#PWR0123"  Part="1"
+F 0 "#PWR0123" H 8400 3900 50  0001 C CNN
 F 1 "VBUS" H 8415 4223 50  0000 C CNN
 F 2 "" H 8400 4050 50  0001 C CNN
@@
 AR Path="/5CDA5615/5CE7F8D4" Ref="#PWR?"  Part="1"
 AR Path="/5CDCD2BF/5CE7F8D4" Ref="#PWR?"  Part="1"
-AR Path="/5D4DF0EE/5CE7F8D4" Ref="#PWR0108"  Part="1"
-F 0 "#PWR0108" H 5800 4200 50  0001 C CNN
+AR Path="/5D4DF0EE/5CE7F8D4" Ref="#PWR0124"  Part="1"
+F 0 "#PWR0124" H 5800 4200 50  0001 C CNN
 F 1 "GND" H 5805 4277 50  0000 C CNN
 F 2 "" H 5800 4450 50  0001 C CNN
@@
 AR Path="/5CDA5615/5CE7F8E1" Ref="#PWR?"  Part="1"
 AR Path="/5CDCD2BF/5CE7F8E1" Ref="#PWR?"  Part="1"
-AR Path="/5D4DF0EE/5CE7F8E1" Ref="#PWR0109"  Part="1"
-F 0 "#PWR0109" H 5100 4200 50  0001 C CNN
+AR Path="/5D4DF0EE/5CE7F8E1" Ref="#PWR0125"  Part="1"
+F 0 "#PWR0125" H 5100 4200 50  0001 C CNN
 F 1 "GND" H 5105 4277 50  0000 C CNN
 F 2 "" H 5100 4450 50  0001 C CNN
@@
 AR Path="/5CDA5615/5CE7F8E7" Ref="#PWR?"  Part="1"
 AR Path="/5CDCD2BF/5CE7F8E7" Ref="#PWR?"  Part="1"
-AR Path="/5D4DF0EE/5CE7F8E7" Ref="#PWR0110"  Part="1"
-F 0 "#PWR0110" H 4400 4200 50  0001 C CNN
+AR Path="/5D4DF0EE/5CE7F8E7" Ref="#PWR0126"  Part="1"
+F 0 "#PWR0126" H 4400 4200 50  0001 C CNN
 F 1 "GND" H 4405 4277 50  0000 C CNN
 F 2 "" H 4400 4450 50  0001 C CNN
@@
 AR Path="/5CDA5615/5CE7F8F0" Ref="#PWR?"  Part="1"
 AR Path="/5CDCD2BF/5CE7F8F0" Ref="#PWR?"  Part="1"
-AR Path="/5D4DF0EE/5CE7F8F0" Ref="#PWR0111"  Part="1"
-F 0 "#PWR0111" H 4150 4200 50  0001 C CNN
+AR Path="/5D4DF0EE/5CE7F8F0" Ref="#PWR0127"  Part="1"
+F 0 "#PWR0127" H 4150 4200 50  0001 C CNN
 F 1 "GND" H 4155 4277 50  0000 C CNN
 F 2 "" H 4150 4450 50  0001 C CNN
@@
 AR Path="/5CDA5615/5CE7F8F6" Ref="R?"  Part="1"
 AR Path="/5CDCD2BF/5CE7F8F6" Ref="R?"  Part="1"
-AR Path="/5D4DF0EE/5CE7F8F6" Ref="R15"  Part="1"
-F 0 "R15" V 4145 4100 50  0000 C CNN
+AR Path="/5D4DF0EE/5CE7F8F6" Ref="R17"  Part="1"
+F 0 "R17" V 4145 4100 50  0000 C CNN
 F 1 "82k" V 4236 4100 50  0000 C CNN
 F 2 "Resistor_SMD:R_0603_1608Metric" V 4390 4090 50  0001 C CNN
@@
 AR Path="/5CDA5615/5CE7F8FF" Ref="#PWR?"  Part="1"
 AR Path="/5CDCD2BF/5CE7F8FF" Ref="#PWR?"  Part="1"
-AR Path="/5D4DF0EE/5CE7F8FF" Ref="#PWR0112"  Part="1"
-F 0 "#PWR0112" H 3200 2500 50  0001 C CNN
+AR Path="/5D4DF0EE/5CE7F8FF" Ref="#PWR0128"  Part="1"
+F 0 "#PWR0128" H 3200 2500 50  0001 C CNN
 F 1 "+5V" H 3215 2823 50  0000 C CNN
 F 2 "" H 3200 2650 50  0001 C CNN
@@
 AR Path="/5CDA5615/5CE7F916" Ref="#PWR?"  Part="1"
 AR Path="/5CDCD2BF/5CE7F916" Ref="#PWR?"  Part="1"
-AR Path="/5D4DF0EE/5CE7F916" Ref="#PWR0113"  Part="1"
-F 0 "#PWR0113" H 3200 2800 50  0001 C CNN
+AR Path="/5D4DF0EE/5CE7F916" Ref="#PWR0129"  Part="1"
+F 0 "#PWR0129" H 3200 2800 50  0001 C CNN
 F 1 "GND" H 3205 2877 50  0000 C CNN
 F 2 "" H 3200 3050 50  0001 C CNN
@@
 AR Path="/5CDA5615/5CE7F91C" Ref="#PWR?"  Part="1"
 AR Path="/5CDCD2BF/5CE7F91C" Ref="#PWR?"  Part="1"
-AR Path="/5D4DF0EE/5CE7F91C" Ref="#PWR0114"  Part="1"
-F 0 "#PWR0114" H 3600 2800 50  0001 C CNN
+AR Path="/5D4DF0EE/5CE7F91C" Ref="#PWR0130"  Part="1"
+F 0 "#PWR0130" H 3600 2800 50  0001 C CNN
 F 1 "GND" H 3605 2877 50  0000 C CNN
 F 2 "" H 3600 3050 50  0001 C CNN
@@
 P 3700 3600
 AR Path="/5CDA5615/5CE7F930" Ref="R?"  Part="1"
-AR Path="/5D4DF0EE/5CE7F930" Ref="R14"  Part="1"
-F 0 "R14" V 3900 3550 50  0000 L CNN
+AR Path="/5D4DF0EE/5CE7F930" Ref="R16"  Part="1"
+F 0 "R16" V 3900 3550 50  0000 L CNN
 F 1 "10k" V 3800 3500 50  0000 L CNN
 F 2 "Resistor_SMD:R_0603_1608Metric" V 3740 3590 50  0001 C CNN
@@
 P 3500 3600
 AR Path="/5CDA5615/5CE7F936" Ref="#PWR?"  Part="1"
-AR Path="/5D4DF0EE/5CE7F936" Ref="#PWR0115"  Part="1"
-F 0 "#PWR0115" H 3500 3450 50  0001 C CNN
+AR Path="/5D4DF0EE/5CE7F936" Ref="#PWR0131"  Part="1"
+F 0 "#PWR0131" H 3500 3450 50  0001 C CNN
 F 1 "+5V" H 3515 3773 50  0000 C CNN
 F 2 "" H 3500 3600 50  0001 C CNN
@@
 Wire Wire Line
 	3500 3600 3550 3600
-Wire Wire Line
-	4250 3700 4550 3700
 Wire Wire Line
 	3850 3600 4550 3600
@@
 AR Path="/5CDA5615/5CE7F957" Ref="#PWR?"  Part="1"
 AR Path="/5CDCD2BF/5CE7F957" Ref="#PWR?"  Part="1"
-AR Path="/5D4DF0EE/5CE7F957" Ref="#PWR0116"  Part="1"
-F 0 "#PWR0116" H 5850 2300 50  0001 C CNN
+AR Path="/5D4DF0EE/5CE7F957" Ref="#PWR0132"  Part="1"
+F 0 "#PWR0132" H 5850 2300 50  0001 C CNN
 F 1 "VBUS" H 5865 2623 50  0000 C CNN
 F 2 "" H 5850 2450 50  0001 C CNN
@@
 	1    0    0    -1
 $EndComp
+$Comp
+L Device:R_US R15
+U 1 1 5CECE4CD
+P 3300 3700
+F 0 "R15" V 3095 3700 50  0000 C CNN
+F 1 "27k" V 3186 3700 50  0000 C CNN
+F 2 "Resistor_SMD:R_0603_1608Metric" V 3340 3690 50  0001 C CNN
+F 3 "~" H 3300 3700 50  0001 C CNN
+	1    3300 3700
+	0    1    1    0
+$EndComp
+Wire Wire Line
+	3450 3700 4550 3700
+$Comp
+L power:VBUS #PWR0133
+U 1 1 5CED0B3D
+P 3050 3550
+F 0 "#PWR0133" H 3050 3400 50  0001 C CNN
+F 1 "VBUS" H 3065 3723 50  0000 C CNN
+F 2 "" H 3050 3550 50  0001 C CNN
+F 3 "" H 3050 3550 50  0001 C CNN
+	1    3050 3550
+	1    0    0    -1
+$EndComp
+Wire Wire Line
+	3050 3550 3050 3700
+Wire Wire Line
+	3050 3700 3150 3700
 $EndSCHEMATC
