File: bumblebee-addon/bumblebee-addon.sch (KiCad schematic (older format))
At the start: 16 parts

Commit message: Started work on bumblebee-addon
Parts:
- removed D?: LED, LED_SMD:LED_0603_1608Metric, symbol Device:LED
- removed R?: 1k, Resistor_SMD:R_0603_1608Metric, symbol Device:R_US
- removed U? (x2): MCP4922-ESL, symbol Analog_DAC:MCP4922-ESL
- added C3: 0.1u, Capacitor_SMD:C_0603_1608Metric, symbol Device:C_Small
- added C4, C5: 0.1u, Capacitor_SMD:C_0603_1608Metric, symbol Device:C
- added J5: FTDI_FLASH, Connector_PinSocket_2.54mm:PinSocket_1x06_P2.54mm_Vertical, symbol Connector_Generic:Conn_01x06
- added J6: INTERFACE, Connector_JST:JST_XH_B8B-XH-A_1x08_P2.50mm_Vertical, symbol Connector_Generic:Conn_01x08
- added U2, U3: MCP4902, Package_SO:SOIC-14_3.9x8.7mm_P1.27mm, symbol Analog_DAC:MCP4902
- J1: renamed from J?; footprint (none) -> Connector_RJ:RJ12_Amphenol_54601
- J2: renamed from J?; footprint footprints:TerminalBlock_TE_282834-4_1x04_P2.54mm_Horizontal -> Connector_JST:JST_XH_B4B-XH-A_1x04_P2.50mm_Vertical
- J3: renamed from J?; footprint footprints:TerminalBlock_TE_282834-8_1x08_P2.54mm_Horizontal -> Connector_JST:JST_XH_B8B-XH-A_1x08_P2.50mm_Vertical
- RV1: renamed from RV?; footprint footprints:Potentiometer_Bourns_PTV09A-1_Single_Vertical -> Potentiometer_THT:Potentiometer_Bourns_PTV09A-1_Single_Vertical
- U1: renamed from U?; symbol Bumblebee-dual-motor-driver-rescue:ATmega328P-AU-MCU_Microchip_ATmega-interface-board-rescue -> bumblebee-addon-rescue:ATmega328P-AU-MCU_Microchip_ATmega-interface-board-rescue-Bumblebee-dual-motor-driver-rescue
- gave numbers to parts that had none: 7
Connections:
- net NTC2 is gone; now on net JS_DETECT: U1.24 (PC1)
- net +3V3: now also C1.1, C2.1, J2.1 (Pin_1), J4.2 (Pin_2), R1.1, RV1.3, U1.18 (AVCC), U1.4 (VCC), U1.6 (VCC), C4.1, C5.1, J5.3 (Pin_3), J6.1 (Pin_1), J6.2 (Pin_2), J6.5 (Pin_5), U2.1 (Vdd), U2.11 (VrefB), U2.13 (VrefA), U3.1 (Vdd), U3.11 (VrefB), U3.13 (VrefA)
- net GND: now also C4.2, C5.2, J5.1 (Pin_1), J6.8 (Pin_8), U2.12 (Vss), U3.12 (Vss)
- net MOSI: now also U2.5 (SDI), U3.5 (SDI)
- net RESET: now also C3.2
- net SCK: now also U2.4 (SCK), U3.4 (SCK)
- removed net +5V: C1.1, C2.1, J2.1 (Pin_1), J4.2 (Pin_2), R1.1, RV1.3, U1.18 (AVCC), U1.20 (AREF), U1.4 (VCC), U1.6 (VCC)
- net M8RXD renamed FTDI_TX
- net FTDI_TX: now also J5.4 (Pin_4)
- net M8TXD renamed FTDI_RX
- net FTDI_RX: now also J5.5 (Pin_5)
- net MOTOR1_DIR renamed DAC1_LDAC
- net DAC1_LDAC: now also U2.8 (~LDAC)
- net MOTOR1_PWM renamed DAC1_CS
- net DAC1_CS: now also U2.3 (~CS)
- net MOTOR2_DIR renamed DAC2_LDAC
- net DAC2_LDAC: now also U3.8 (~LDAC)
- net MOTOR2_PWM renamed DAC2_CS
- net DAC2_CS: now also U3.3 (~CS)
- net NTC1: no longer names the net of U1.25 (PC2)
- new net FTDI_DTR: C3.1, J5.6 (Pin_6)
- new net L_BLACK: J6.3 (Pin_3), U2.10 (VB)
- new net L_GREEN: J6.4 (Pin_4), U2.14 (VA)
- new net R_BLACK: J6.6 (Pin_6), U3.10 (VB)
- new net R_GREEN: J6.7 (Pin_7), U3.14 (VA)
Other:
- note added: "FTDI_PROG"
- note added: "Fine to program at 5V, as long as it isn't\nalso plugged into the motor driver board."
- note added: "JS Input"
- note added: "Output"
- note added: "Status LED"
- note removed: "Status LEDs"
- moved on the sheet: D1, J1, J2, J3, R2

Commit message: Shipped new revs of all boards.
Parts:
- J2: footprint Connector_JST:JST_XH_B4B-XH-A_1x04_P2.50mm_Vertical -> footprints:TerminalBlock_TE_282834-4_1x04_P2.54mm_Horizontal
- J3: footprint Connector_JST:JST_XH_B8B-XH-A_1x08_P2.50mm_Vertical -> footprints:TerminalBlock_TE_282834-8_1x08_P2.54mm_Horizontal
- RV1: footprint Potentiometer_THT:Potentiometer_Bourns_PTV09A-1_Single_Vertical -> footprints:Potentiometer_Bourns_PTV09A-1_Single_Vertical
Connections:
- net BTN_DN: now also J3.6 (Pin_6); no longer J3.3 (Pin_3)
- net BTN_L: now also J3.4 (Pin_4); no longer J3.5 (Pin_5)
- net BTN_R: now also J3.2 (Pin_2); no longer J3.7 (Pin_7)
- net BTN_UP: now also J3.8 (Pin_8); no longer J3.1 (Pin_1)
- net GND: now also J3.1 (Pin_1), J3.3 (Pin_3), J3.5 (Pin_5), J3.7 (Pin_7); no longer J3.2 (Pin_2), J3.4 (Pin_4), J3.6 (Pin_6), J3.8 (Pin_8)
Changed lines of the file:
@@
 F 0 "RV1" H 3282 2104 50  0000 R CNN
 F 1 "R_POT_US" H 3282 2195 50  0000 R CNN
-F 2 "Potentiometer_THT:Potentiometer_Bourns_PTV09A-1_Single_Vertical" H 3350 2150 50  0001 C CNN
+F 2 "footprints:Potentiometer_Bourns_PTV09A-1_Single_Vertical" H 3350 2150 50  0001 C CNN
 F 3 "~" H 3350 2150 50  0001 C CNN
 	1    3350 2150
@@
 F 0 "J2" H 3300 4700 50  0000 L CNN
 F 1 "HEADER" H 3250 5200 50  0000 L CNN
-F 2 "Connector_JST:JST_XH_B4B-XH-A_1x04_P2.50mm_Vertical" H 3350 5000 50  0001 C CNN
+F 2 "footprints:TerminalBlock_TE_282834-4_1x04_P2.54mm_Horizontal" H 3350 5000 50  0001 C CNN
 F 3 "~" H 3350 5000 50  0001 C CNN
 	1    3350 5000
@@
 Text Label 600  1450 0    50   ~ 0
 JS_Y
-$Comp
-L Connector_Generic:Conn_01x08 J3
-U 1 1 5CECB5F2
-P 3350 6100
-F 0 "J3" H 3300 5600 50  0000 L CNN
-F 1 "HEADER" H 3250 6500 50  0000 L CNN
-F 2 "Connector_JST:JST_XH_B8B-XH-A_1x08_P2.50mm_Vertical" H 3350 6100 50  0001 C CNN
-F 3 "~" H 3350 6100 50  0001 C CNN
-	1    3350 6100
-	1    0    0    -1
-$EndComp
 Text Label 2300 6000 0    50   ~ 0
 BTN_DN
@@
 Wire Wire Line
 	2300 5800 3150 5800
-Wire Wire Line
-	2750 5900 3150 5900
 Wire Wire Line
 	2300 6000 3150 6000
@@
 Wire Wire Line
 	5600 1000 5600 1450
+Wire Wire Line
+	2750 5900 3150 5900
+$Comp
+L Connector_Generic:Conn_01x08 J3
+U 1 1 5CECB5F2
+P 3350 6200
+F 0 "J3" H 3300 5700 50  0000 L CNN
+F 1 "HEADER" H 3250 6600 50  0000 L CNN
+F 2 "footprints:TerminalBlock_TE_282834-8_1x08_P2.54mm_Horizontal" H 3350 6200 50  0001 C CNN
+F 3 "~" H 3350 6200 50  0001 C CNN
+	1    3350 6200
+	1    0    0    1
+$EndComp
 $EndSCHEMATC
