File: bumblebee-compact-board/pro-mini-adapter-board.kicad_pcb (KiCad board)
At the start: 2 copper layers, 65.4 x 66 mm, 19 parts, among them J1 RMOTOR, J2 LMOTOR, J3 Conn_01x04, J4 JST-XH, J5 Conn_01x04, J6 HEADER, J7 Conn_01x02, SW1 SW_DIP_x04

Commit message: Shipped new revs of all boards.
Parts:
- C2: footprint Capacitor_THT:C_Radial_D8.0mm_H7.0mm_P3.50mm -> Capacitor_THT:CP_Radial_D8.0mm_P3.50mm
Other:
- board text added: "5V F/RV L/R GND"
- board text added: "Willem Hillier revB 5/27/2019"
- board text removed: "5V F/RV L/R 5V"
- board text removed: "Willem Hillier revA 5/11/2019"
